File: Hardware/diagDisplay(0805)_kyleHess2.sch (KiCad schematic (older format))
At the start: 150 parts, among them IC3 74595D, IC5 74595D, IC7 74595D

Commit message: Updated hardware to use latest library references.
Parts:
- IC3, IC5, IC7, R1, R2: footprint diagDisplay(0805)_kyleHess2:SO16 -> Package_SO:SOIC-16_3.9x9.9mm_P1.27mm
- LED1, LED10, LED100, LED101, LED102, LED103, LED104, LED105, LED106, LED107, LED108, LED109, LED11, LED110, LED111, LED112, LED113, LED114, LED115, LED116, LED117, LED118, LED119, LED12, LED120, LED121, LED122, LED123, LED124, LED125, LED126, LED127, LED128, LED13, LED14, LED15, LED16, LED17, LED18, LED19, LED2, LED20, LED21, LED22, LED23, LED24, LED25, LED26, LED27, LED28, LED29, LED3, LED30, LED31, LED32, LED33, LED34, LED35, LED36, LED37, LED38, LED39, LED4, LED40, LED41, LED42, LED43, LED44, LED45, LED46, LED47, LED48, LED49, LED5, LED50, LED51, LED52, LED53, LED54, LED55, LED56, LED57, LED58, LED59, LED6, LED60, LED61, LED62, LED63, LED64, LED65, LED66, LED67, LED68, LED69, LED7, LED70, LED71, LED72, LED73, LED74, LED75, LED76, LED77, LED78, LED79, LED8, LED80, LED81, LED82, LED83, LED84, LED85, LED86, LED87, LED88, LED89, LED9, LED90, LED91, LED92, LED93, LED94, LED95, LED96, LED97, LED98, LED99: footprint diagDisplay(0805)_kyleHess2:CHIPLED_0805 -> LED_SMD:LED_0805_2012Metric
- R10, R3, R4, R5, R6, R7, R8, R9: footprint diagDisplay(0805)_kyleHess2:M0805 -> Resistor_SMD:R_0805_2012Metric
- U$1, U$2, U$3, U$4, U$5, U$6, U$7, U$8: footprint diagDisplay(0805)_kyleHess2:SOT23-3 -> Package_TO_SOT_SMD:SOT-23
